File: ripple_glaettung.kicad_pcb (KiCad board)
At the start: 2 copper layers, 57.1 x 27.9 mm, 12 parts, among them J1 , J2 , Q1 MJE3055T

Commit message: fine tuning pcb picture
Parts:
- removed  : , MountingHole:MountingHole_2.7mm (x4)
- added HS1: Heatsink, Heatsink:Heatsink_Fischer_SK129-STS_42x25mm_2xDrill2.5mm, F.Cu at (138.5, 89.4)
- J1, J2: value (none) -> Screw_Terminal_01x02
- Q1: value MJE3055T -> TIP142; footprint digikey-footprints:TO-220-3 -> Package_TO_SOT_THT:TO-218-3_Vertical
- moved C1 65.5 mm to (133.4, 114.8)
- moved R1 65.5 mm to (133.4, 105.9)
- moved C2 65.5 mm to (148.6, 119.9)
- moved C3 65.5 mm to (146.1, 111.0)
- moved C4 65.5 mm to (152.4, 111.0)
- moved J1 65.5 mm to (115.6, 116.1)
- moved J2 65.5 mm to (161.3, 111.0)
- moved Q1 53.7 mm to (133.0, 94.0)
Routing:
- net VCC: track 33.0 -> 65.3 mm
- net Net-(C1-Pad1): track 42.9 -> 52.4 mm
- net Net-(J2-Pad1): track 17.9 -> 24.4 mm
- net (no net): vias 0 -> 4
Other:
- board size 57.1 x 27.9 mm -> 57 x 52 mm
- board text added: "voltage ripple suppressor"
